Commit message: 头部相机标定完毕

File: src/qi_robot_description/urdf/s4_40DOF_fullbody_with_handeye_camera.urdf (robot description, URDF)
Before this commit: robot S4_40DOF, 52 links, 51 joints
Links:
- added link head_calibrated_camera_color_optical_frame; visual box size=0.090 0.025 0.025; visual cylinder length=0.003 radius=0.0045
- added link left_calibrated_camera_color_optical_frame; visual box size=0.042 0.042 0.023; visual cylinder length=0.003 radius=0.0045
- link base_link: geometry collision box size=0.25 0.20 0.12
- link calibrated_camera_color_optical_frame: geometry visual box size=0.042 0.042 0.023; visual cylinder length=0.003 radius=0.0045
Joints:
- added joint LH_hand_to_calibrated_camera: type fixed, parent LH_hand_base_link, child left_calibrated_camera_color_optical_frame, origin xyz=-0.0209877889 -0.0745941356 0.0914989107 rpy=-0.3853061096 0.8654732231 -0.0927412477
- added joint base_to_head_calibrated_camera: type fixed, parent base_link, child head_calibrated_camera_color_optical_frame, origin xyz=0.0240925853 0.0044939526 0.6924775167 rpy=-2.3896833190 0.0485398982 -1.5644776018
